File: PCB_glove/PCB_glove.kicad_sch (KiCad schematic)
At the start: 0 parts

Commit message: Add rough schematic draft checkpoint
Parts:
- added J1: STM32N6570-DK FUNCTIONAL INTERFACE PLACEHOLDER, symbol Connector_Generic:Conn_01x18
- added J2: THUMB REMOTE IMU CONNECTOR TBD, symbol Connector_Generic:Conn_01x09
- added J3: INDEX REMOTE IMU CONNECTOR TBD, symbol Connector_Generic:Conn_01x09
- added J4: MIDDLE REMOTE IMU CONNECTOR TBD, symbol Connector_Generic:Conn_01x09
- added J5: RING REMOTE IMU CONNECTOR TBD, symbol Connector_Generic:Conn_01x09
- added J6: PINKY REMOTE IMU CONNECTOR TBD, symbol Connector_Generic:Conn_01x09
- added J7: PROTECTED 5V BENCH INPUT TBD, symbol Connector_Generic:Conn_01x02
Connections:
- new net +3V3_IMU_TBD: J2.2 (Pin_2), J3.2 (Pin_2), J4.2 (Pin_2), J5.2 (Pin_2), J6.2 (Pin_2)
- new net DK_3V3_ACCESS_TBD: J1.2 (Pin_2)
- new net DK_5V_ACCESS_TBD: J1.1 (Pin_1)
- new net DK_SPARE_TBD: J1.18 (Pin_18)
- new net GND: J1.17 (Pin_17), J1.3 (Pin_3), J2.1 (Pin_1), J2.3 (Pin_3), J3.1 (Pin_1), J3.3 (Pin_3), J4.1 (Pin_1), J4.3 (Pin_3), J5.1 (Pin_1), J5.3 (Pin_3), J6.1 (Pin_1), J6.3 (Pin_3), J7.2 (Pin_2)
- new net IMU_INDEX_CS_N: J1.8 (Pin_8), J3.7 (Pin_7)
- new net IMU_INDEX_INT1: J1.13 (Pin_13), J3.8 (Pin_8)
- new net IMU_INDEX_INT2_TBD: J3.9 (Pin_9)
- new net IMU_MIDDLE_CS_N: J1.9 (Pin_9), J4.7 (Pin_7)
- new net IMU_MIDDLE_INT1: J1.14 (Pin_14), J4.8 (Pin_8)
- new net IMU_MIDDLE_INT2_TBD: J4.9 (Pin_9)
- new net IMU_PINKY_CS_N: J1.11 (Pin_11), J6.7 (Pin_7)
- new net IMU_PINKY_INT1: J1.16 (Pin_16), J6.8 (Pin_8)
- new net IMU_PINKY_INT2_TBD: J6.9 (Pin_9)
- new net IMU_RING_CS_N: J1.10 (Pin_10), J5.7 (Pin_7)
- new net IMU_RING_INT1: J1.15 (Pin_15), J5.8 (Pin_8)
- new net IMU_RING_INT2_TBD: J5.9 (Pin_9)
- new net IMU_SPI_MISO: J1.6 (Pin_6), J2.6 (Pin_6), J3.6 (Pin_6), J4.6 (Pin_6), J5.6 (Pin_6), J6.6 (Pin_6)
- new net IMU_SPI_MOSI: J1.5 (Pin_5), J2.5 (Pin_5), J3.5 (Pin_5), J4.5 (Pin_5), J5.5 (Pin_5), J6.5 (Pin_5)
- new net IMU_SPI_SCK: J1.4 (Pin_4), J2.4 (Pin_4), J3.4 (Pin_4), J4.4 (Pin_4), J5.4 (Pin_4), J6.4 (Pin_4)
- new net IMU_THUMB_CS_N: J1.7 (Pin_7), J2.7 (Pin_7)
- new net IMU_THUMB_INT1: J1.12 (Pin_12), J2.8 (Pin_8)
- new net IMU_THUMB_INT2_TBD: J2.9 (Pin_9)
- new net VIN_5V_PROVISIONAL: J7.1 (Pin_1)
Other:
- note added: "+3V3_IMU_TBD is intentionally not driven in this draft pending DK/power-budget documentation."
- note added: "CAMERA 1 PLACEHOLDER / TBD ONLY"
- note added: "CAMERA 2 PLACEHOLDER / TBD ONLY"
- note added: "CAMERA CIRCUIT BLOCKED PENDING DOCUMENTATION"
- note added: "CONNECTOR MPN/FOOTPRINT TBD"
- note added: "DK PIN MAPPING TBD"
- note added: "DK interface reservation: shared SPI + five CS_N + five INT1. Exact DK connector/header, MCU pins, voltage domain, solder bridges, and conflicts remain TBD."
- note added: "DRAFT ONLY"
- note added: "Each remote finger module is provisional ISM330DHCX. The separate sensor PCB is not part of this central adapter schematic."
- note added: "FUNCTIONAL NET NAMES ONLY — J1 PIN NUMBERS DO NOT REPRESENT STM32N6570-DK HEADER POSITIONS."
- note added: "Finger connector pin order is a logical draft only: 1 GND, 2 +3V3_IMU_TBD, 3 GND, 4 SCK, 5 MOSI, 6 MISO, 7 CS_N, 8 INT1, 9 INT2_TBD."
- note added: "INT2 is reserved at each logical finger interface but is not mapped to the DK in this draft."
- note added: "NOT FOR FABRICATION"
- note added: "No connector, pinout, rails, clock, control bus, reset, data lanes, protection, footprint, or wiring defined."
- note added: "PCB_glove — STM32N6570-DK ADAPTER / FIVE-FINGER SENSOR INTERFACE"
- note added: "POWER PLACEHOLDER"
- note added: "Provisional protected wired 5 V entry only. Protection, regulator, current limit, rail source, sequencing, test points, connector MPN, and footprints are TBD."
- note added: "RUN FULL REVIEW BEFORE PCB LAYOUT"
- note added: "Reference-design lesson retained: local IMU VDD/VDDIO decoupling and short return paths are required; exact values and implementation require current datasheet review."
- note added: "SHARED SPI HARNESS DRAFT: reserve source-series damping options on SCK/MOSI and per-branch review; values/footprints TBD after cable measurements."
- note added: "TODO BEFORE REVIEW: prove DK mapping; select connectors; verify ISM330DHCX and SPI reset behavior; complete power budget; obtain camera documentation; run ERC after pin types are finalized."
- note added: "This schematic is incomplete and unverified. It does not authorize PCB layout, routing, procurement, assembly, or fabrication."

Commit message: Add audited schematic draft and local draft libraries
Parts:
- removed J1: STM32N6570-DK FUNCTIONAL INTERFACE PLACEHOLDER, symbol Connector_Generic:Conn_01x18
- removed J2: THUMB REMOTE IMU CONNECTOR TBD, symbol Connector_Generic:Conn_01x09
- removed J3: INDEX REMOTE IMU CONNECTOR TBD, symbol Connector_Generic:Conn_01x09
- removed J4: MIDDLE REMOTE IMU CONNECTOR TBD, symbol Connector_Generic:Conn_01x09
- removed J5: RING REMOTE IMU CONNECTOR TBD, symbol Connector_Generic:Conn_01x09
- removed J6: PINKY REMOTE IMU CONNECTOR TBD, symbol Connector_Generic:Conn_01x09
- removed J7: PROTECTED 5V BENCH INPUT TBD, symbol Connector_Generic:Conn_01x02
Other:
- added sheet CAMERA PLACEHOLDERS (camera_placeholders.kicad_sch)
- added sheet DK ADAPTER HEADERS (dk_adapter_headers.kicad_sch)
- added sheet FINGER IMU MODULE REFERENCE (finger_imu_module_reference.kicad_sch)
- added sheet IMU CENTRAL DISTRIBUTION (imu_central_distribution.kicad_sch)
- added sheet NOTES AND TODOS (notes_and_todos.kicad_sch)
- added sheet POWER AND TEST (power_and_test.kicad_sch)
- note added: "Global logical net names connect the detailed sheets. Physical DK pins, production connectors, power architecture, and camera implementation remain blocked/TBD."
- note added: "No PCB layout, routing, fabrication output, final footprint, or verified camera circuit is authorized by this schematic package."
- note added: "PCB_glove — DETAILED SCHEMATIC PREPARATION OVERVIEW"
- note added: "STM32N6570-DK is the host. This project is an adapter/interface/sensor draft — not a bare STM32N6 controller."
- note removed: "+3V3_IMU_TBD is intentionally not driven in this draft pending DK/power-budget documentation."
- note removed: "CAMERA 1 PLACEHOLDER / TBD ONLY"
- note removed: "CAMERA 2 PLACEHOLDER / TBD ONLY"
- note removed: "DK interface reservation: shared SPI + five CS_N + five INT1. Exact DK connector/header, MCU pins, voltage domain, solder bridges, and conflicts remain TBD."
- note removed: "Each remote finger module is provisional ISM330DHCX. The separate sensor PCB is not part of this central adapter schematic."
- note removed: "FUNCTIONAL NET NAMES ONLY — J1 PIN NUMBERS DO NOT REPRESENT STM32N6570-DK HEADER POSITIONS."
- note removed: "Finger connector pin order is a logical draft only: 1 GND, 2 +3V3_IMU_TBD, 3 GND, 4 SCK, 5 MOSI, 6 MISO, 7 CS_N, 8 INT1, 9 INT2_TBD."
- note removed: "INT2 is reserved at each logical finger interface but is not mapped to the DK in this draft."
- note removed: "No connector, pinout, rails, clock, control bus, reset, data lanes, protection, footprint, or wiring defined."
- note removed: "PCB_glove — STM32N6570-DK ADAPTER / FIVE-FINGER SENSOR INTERFACE"
- note removed: "POWER PLACEHOLDER"
- note removed: "Provisional protected wired 5 V entry only. Protection, regulator, current limit, rail source, sequencing, test points, connector MPN, and footprints are TBD."
- note removed: "Reference-design lesson retained: local IMU VDD/VDDIO decoupling and short return paths are required; exact values and implementation require current datasheet review."
- note removed: "SHARED SPI HARNESS DRAFT: reserve source-series damping options on SCK/MOSI and per-branch review; values/footprints TBD after cable measurements."
- note removed: "TODO BEFORE REVIEW: prove DK mapping; select connectors; verify ISM330DHCX and SPI reset behavior; complete power budget; obtain camera documentation; run ERC after pin types are finalized."
- note removed: "This schematic is incomplete and unverified. It does not authorize PCB layout, routing, procurement, assembly, or fabrication."
