File: PCB_glove/imu_central_distribution.kicad_sch (KiCad schematic)
At the start: 17 parts, among them J2 THUMB_IMU — 9-POS LOGICAL CON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, J3 INDEX_IMU — 9-POS LOGICAL CON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, J4 MIDDLE_IMU — 9-POS LOGICAL CO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, J5 RING_IMU — 9-POS LOGICAL CONN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, J6 PINKY_IMU — 9-POS LOGICAL CON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

Commit message: all
Connections:
- net IMU_INDEX_INT2_TBD: no longer names the net of J3.9 (Pin_9)
- net IMU_MIDDLE_INT2_TBD: no longer names the net of J4.9 (Pin_9)
- net IMU_PINKY_INT2_TBD: no longer names the net of J6.9 (Pin_9)
- net IMU_RING_INT2_TBD: no longer names the net of J5.9 (Pin_9)
- net IMU_THUMB_INT2_TBD: no longer names the net of J2.9 (Pin_9)
- no-connect marks 0 -> 5
Other:
- note added: "DK_IMU_SPI_SCK_TBD and DK_IMU_SPI_MOSI_TBD are DK-side series-option nets; the physical DK pins are proven, while R1/R2 values remain deferred pending signal-integrity testing."
- note added: "INDEX_IMU LOGICAL TABLE: 1 GND | 2 +3V3_IMU | 3 GND | 4 SCK | 5 MOSI | 6 MISO | 7 CS_N | 8 INT1 | 9 INT2 DNC FOR V1"
- note added: "INT1 is direct per finger. INT2 is deliberately not connected for v1. Two ground contacts are retained in the logical connector budget."
- note added: "MIDDLE_IMU LOGICAL TABLE: 1 GND | 2 +3V3_IMU | 3 GND | 4 SCK | 5 MOSI | 6 MISO | 7 CS_N | 8 INT1 | 9 INT2 DNC FOR V1"
- note added: "PINKY_IMU LOGICAL TABLE: 1 GND | 2 +3V3_IMU | 3 GND | 4 SCK | 5 MOSI | 6 MISO | 7 CS_N | 8 INT1 | 9 INT2 DNC FOR V1"
- note added: "RING_IMU LOGICAL TABLE: 1 GND | 2 +3V3_IMU | 3 GND | 4 SCK | 5 MOSI | 6 MISO | 7 CS_N | 8 INT1 | 9 INT2 DNC FOR V1"
- note added: "THUMB_IMU LOGICAL TABLE: 1 GND | 2 +3V3_IMU | 3 GND | 4 SCK | 5 MOSI | 6 MISO | 7 CS_N | 8 INT1 | 9 INT2 DNC FOR V1"
- note removed: "DK_IMU_SPI_SCK_TBD and DK_IMU_SPI_MOSI_TBD are the unverified DK-side nets; R1/R2 separate them from the conditioned harness buses."
- note removed: "INDEX_IMU LOGICAL TABLE: 1 GND | 2 +3V3_IMU | 3 GND | 4 SCK | 5 MOSI | 6 MISO | 7 CS_N | 8 INT1 | 9 INT2/NC TBD"
- note removed: "INT1 is direct per finger. INT2 remains optional/TBD. Two ground contacts are retained in the logical connector budget."
- note removed: "MIDDLE_IMU LOGICAL TABLE: 1 GND | 2 +3V3_IMU | 3 GND | 4 SCK | 5 MOSI | 6 MISO | 7 CS_N | 8 INT1 | 9 INT2/NC TBD"
- note removed: "PINKY_IMU LOGICAL TABLE: 1 GND | 2 +3V3_IMU | 3 GND | 4 SCK | 5 MOSI | 6 MISO | 7 CS_N | 8 INT1 | 9 INT2/NC TBD"
- note removed: "RING_IMU LOGICAL TABLE: 1 GND | 2 +3V3_IMU | 3 GND | 4 SCK | 5 MOSI | 6 MISO | 7 CS_N | 8 INT1 | 9 INT2/NC TBD"
- note removed: "THUMB_IMU LOGICAL TABLE: 1 GND | 2 +3V3_IMU | 3 GND | 4 SCK | 5 MOSI | 6 MISO | 7 CS_N | 8 INT1 | 9 INT2/NC TBD"
Changed lines of the file:
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@@
     (effects (font (size 1.27 1.27)) (justify left))
   )
-  (wire (pts (xy 35.56 142.24) (xy 40.64 142.24)) (stroke (width 0) (type default)))
-  (global_label "IMU_THUMB_INT2_TBD" (shape bidirectional) (at 40.64 142.24 0) (fields_autoplaced)
-    (effects (font (size 1.27 1.27)) (justify left))
-  )
-  (text "THUMB_IMU LOGICAL TABLE: 1 GND | 2 +3V3_IMU | 3 GND | 4 SCK | 5 MOSI | 6 MISO | 7 CS_N | 8 INT1 | 9 INT2/NC TBD" (at 17.78 177.8 0)
+  (no_connect (at 35.56 142.24))
+  (text "THUMB_IMU LOGICAL TABLE: 1 GND | 2 +3V3_IMU | 3 GND | 4 SCK | 5 MOSI | 6 MISO | 7 CS_N | 8 INT1 | 9 INT2 DNC FOR V1" (at 17.78 177.8 0)
     (effects (font (size 0.95 0.95)) (justify left bottom))
   )
@@
     (effects (font (size 1.27 1.27)) (justify left))
   )
-  (wire (pts (xy 111.76 142.24) (xy 116.84 142.24)) (stroke (width 0) (type default)))
-  (global_label "IMU_INDEX_INT2_TBD" (shape bidirectional) (at 116.84 142.24 0) (fields_autoplaced)
-    (effects (font (size 1.27 1.27)) (justify left))
-  )
-  (text "INDEX_IMU LOGICAL TABLE: 1 GND | 2 +3V3_IMU | 3 GND | 4 SCK | 5 MOSI | 6 MISO | 7 CS_N | 8 INT1 | 9 INT2/NC TBD" (at 93.98 177.8 0)
+  (no_connect (at 111.76 142.24))
+  (text "INDEX_IMU LOGICAL TABLE: 1 GND | 2 +3V3_IMU | 3 GND | 4 SCK | 5 MOSI | 6 MISO | 7 CS_N | 8 INT1 | 9 INT2 DNC FOR V1" (at 93.98 177.8 0)
     (effects (font (size 0.95 0.95)) (justify left bottom))
   )
@@
     (effects (font (size 1.27 1.27)) (justify left))
   )
-  (wire (pts (xy 187.96 142.24) (xy 193.04 142.24)) (stroke (width 0) (type default)))
-  (global_label "IMU_MIDDLE_INT2_TBD" (shape bidirectional) (at 193.04 142.24 0) (fields_autoplaced)
-    (effects (font (size 1.27 1.27)) (justify left))
-  )
-  (text "MIDDLE_IMU LOGICAL TABLE: 1 GND | 2 +3V3_IMU | 3 GND | 4 SCK | 5 MOSI | 6 MISO | 7 CS_N | 8 INT1 | 9 INT2/NC TBD" (at 170.18 177.8 0)
+  (no_connect (at 187.96 142.24))
+  (text "MIDDLE_IMU LOGICAL TABLE: 1 GND | 2 +3V3_IMU | 3 GND | 4 SCK | 5 MOSI | 6 MISO | 7 CS_N | 8 INT1 | 9 INT2 DNC FOR V1" (at 170.18 177.8 0)
     (effects (font (size 0.95 0.95)) (justify left bottom))
   )
@@
     (effects (font (size 1.27 1.27)) (justify left))
   )
-  (wire (pts (xy 264.16 142.24) (xy 269.24 142.24)) (stroke (width 0) (type default)))
-  (global_label "IMU_RING_INT2_TBD" (shape bidirectional) (at 269.24 142.24 0) (fields_autoplaced)
-    (effects (font (size 1.27 1.27)) (justify left))
-  )
-  (text "RING_IMU LOGICAL TABLE: 1 GND | 2 +3V3_IMU | 3 GND | 4 SCK | 5 MOSI | 6 MISO | 7 CS_N | 8 INT1 | 9 INT2/NC TBD" (at 246.38 177.8 0)
+  (no_connect (at 264.16 142.24))
+  (text "RING_IMU LOGICAL TABLE: 1 GND | 2 +3V3_IMU | 3 GND | 4 SCK | 5 MOSI | 6 MISO | 7 CS_N | 8 INT1 | 9 INT2 DNC FOR V1" (at 246.38 177.8 0)
     (effects (font (size 0.95 0.95)) (justify left bottom))
   )
@@
     (effects (font (size 1.27 1.27)) (justify left))
   )
-  (wire (pts (xy 340.36 142.24) (xy 345.44 142.24)) (stroke (width 0) (type default)))
-  (global_label "IMU_PINKY_INT2_TBD" (shape bidirectional) (at 345.44 142.24 0) (fields_autoplaced)
-    (effects (font (size 1.27 1.27)) (justify left))
-  )
-  (text "PINKY_IMU LOGICAL TABLE: 1 GND | 2 +3V3_IMU | 3 GND | 4 SCK | 5 MOSI | 6 MISO | 7 CS_N | 8 INT1 | 9 INT2/NC TBD" (at 322.58 177.8 0)
+  (no_connect (at 340.36 142.24))
+  (text "PINKY_IMU LOGICAL TABLE: 1 GND | 2 +3V3_IMU | 3 GND | 4 SCK | 5 MOSI | 6 MISO | 7 CS_N | 8 INT1 | 9 INT2 DNC FOR V1" (at 322.58 177.8 0)
     (effects (font (size 0.95 0.95)) (justify left bottom))
   )
@@
     (effects (font (size 1.27 1.27) (thickness 0.4)) (justify left bottom))
   )
-  (text "INT1 is direct per finger. INT2 remains optional/TBD. Two ground contacts are retained in the logical connector budget." (at 15.24 269.24 0)
+  (text "INT1 is direct per finger. INT2 is deliberately not connected for v1. Two ground contacts are retained in the logical connector budget." (at 15.24 269.24 0)
     (effects (font (size 1.27 1.27)) (justify left bottom))
   )
-  (text "DK_IMU_SPI_SCK_TBD and DK_IMU_SPI_MOSI_TBD are the unverified DK-side nets; R1/R2 separate them from the conditioned harness buses." (at 15.24 276.86 0)
+  (text "DK_IMU_SPI_SCK_TBD and DK_IMU_SPI_MOSI_TBD are DK-side series-option nets; the physical DK pins are proven, while R1/R2 values remain deferred pending signal-integrity testing." (at 15.24 276.86 0)
     (effects (font (size 1.27 1.27)) (justify left bottom))
   )
