File: PCB_glove/dk_adapter_headers.kicad_sch (KiCad schematic)
At the start: 1 part, among them J1 STM32N6570-DK LOGICAL ADAPTER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

Commit message: Add ERC-clean IMU power schematic update
Connections:
- net +3V3_IMU: no longer names the net of J1.3 (Pin_3)
- net +5V_IN_TBD: no longer names the net of J1.1 (Pin_1)
- no-connect marks 2 -> 4
Other:
- note added: "+3V3_IMU is generated locally by the power-sheet LDO. Optional INT2 signals remain reserved but are not finally mapped."
- note added: "DK +5 V IS NOT CONNECTED TO +5V_EXT — DK +3.3 V IS NOT CONNECTED TO +3V3_IMU"
- note added: "DK AND PCB_glove SHARE GND ONLY THROUGH THE DOCUMENTED SIGNAL INTERFACE; POSITIVE POWER RAIL SLOTS ARE NO-CONNECTED."
- note removed: "+3V3_DK_TBD is intentionally no-connected until DK rail headroom and the exact physical header are proven."
- note removed: "+3V3_DK_TBD is observation/access only. Do not assume the DK 3.3 V rail can supply five IMUs."
- note removed: "+3V3_IMU source is defined on the power sheet and remains provisional. Optional INT2 signals are reserved but not mapped."
Changed lines of the file:
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@@
     (pin "24")
   )
-  (wire (pts (xy 55.88 72.39) (xy 60.96 72.39)) (stroke (width 0) (type default)))
-  (global_label "+5V_IN_TBD" (shape bidirectional) (at 60.96 72.39 0) (fields_autoplaced)
-    (effects (font (size 1.27 1.27)) (justify left))
-  )
+  (no_connect (at 55.88 72.39))
   (no_connect (at 55.88 77.47))
-  (wire (pts (xy 55.88 82.55) (xy 60.96 82.55)) (stroke (width 0) (type default)))
-  (global_label "+3V3_IMU" (shape bidirectional) (at 60.96 82.55 0) (fields_autoplaced)
-    (effects (font (size 1.27 1.27)) (justify left))
-  )
+  (no_connect (at 55.88 82.55))
   (wire (pts (xy 55.88 87.63) (xy 60.96 87.63)) (stroke (width 0) (type default)))
   (global_label "GND" (shape bidirectional) (at 60.96 87.63 0) (fields_autoplaced)
@@
     (effects (font (size 1.27 1.27)) (justify left bottom))
   )
-  (text "+3V3_DK_TBD is observation/access only. Do not assume the DK 3.3 V rail can supply five IMUs." (at 15.24 213.36 0)
+  (text "DK +5 V IS NOT CONNECTED TO +5V_EXT — DK +3.3 V IS NOT CONNECTED TO +3V3_IMU" (at 15.24 213.36 0)
     (effects (font (size 1.27 1.27) (thickness 0.4)) (justify left bottom))
   )
-  (text "+3V3_IMU source is defined on the power sheet and remains provisional. Optional INT2 signals are reserved but not mapped." (at 15.24 220.98 0)
+  (text "DK AND PCB_glove SHARE GND ONLY THROUGH THE DOCUMENTED SIGNAL INTERFACE; POSITIVE POWER RAIL SLOTS ARE NO-CONNECTED." (at 15.24 220.98 0)
     (effects (font (size 1.27 1.27)) (justify left bottom))
   )
-  (text "+3V3_DK_TBD is intentionally no-connected until DK rail headroom and the exact physical header are proven." (at 15.24 228.6 0)
+  (text "+3V3_IMU is generated locally by the power-sheet LDO. Optional INT2 signals remain reserved but are not finally mapped." (at 15.24 228.6 0)
     (effects (font (size 1.27 1.27)) (justify left bottom))
   )

Commit message: all
Parts:
- removed J1: STM32N6570-DK LOGICAL ADAPTER HEADER PLACEHOLDER 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, symbol PCB_glove_Draft:DK_LOGICAL_24
- added J10: DK CN7 6-position, symbol PCB_glove_Draft:DK_CN7_6
- added J11: DK CN8 8-position, symbol PCB_glove_Draft:DK_CN8_8
- added J12: DK CN11 8-position, symbol PCB_glove_Draft:DK_CN11_8
- added J13: DK CN12 10-position, symbol PCB_glove_Draft:DK_CN12_10
- added J14: SPI HARNESS, symbol PCB_glove_Draft:HARNESS_1X6
- added J15: CS HARNESS, symbol PCB_glove_Draft:HARNESS_1X6
- added J16: INT HARNESS, symbol PCB_glove_Draft:HARNESS_1X6
- added R18, R19, R20, R21, R22: 10k CS SAFE-STATE PULL-UP, Resistor_SMD:R_0603_1608Metric, symbol PCB_glove_Draft:R_OPTION
Connections:
- net DK_IMU_SPI_MOSI_TBD: now also J13.4 (D11 / PG2)
- net DK_IMU_SPI_SCK_TBD: now also J13.6 (D13 / PE15)
- net GND: now also J11.6 (GND_A), J11.7 (GND_B), J13.7 (GND), J14.2 (CAVITY_2), J14.4 (CAVITY_4), J15.2 (CAVITY_2), J16.2 (CAVITY_2)
- net IMU_INDEX_CS_N: now also J13.2 (D9 / PE14), J15.3 (CAVITY_3), R19.2
- net IMU_INDEX_INT1: now also J12.5 (D4 / PH5), J16.3 (CAVITY_3)
- net IMU_MIDDLE_CS_N: now also J13.1 (D8 / PE7), J15.4 (CAVITY_4), R20.2
- net IMU_MIDDLE_INT1: now also J12.4 (D3 / PE9), J16.4 (CAVITY_4)
- net IMU_PINKY_CS_N: now also J12.7 (D6 / PE13), J15.6 (CAVITY_6), R22.2
- net IMU_PINKY_INT1: now also J10.4 (A3 / PD11), J16.6 (CAVITY_6)
- net IMU_RING_CS_N: now also J12.8 (D7 / PD6), J15.5 (CAVITY_5), R21.2
- net IMU_RING_INT1: now also J12.3 (D2 / PD0), J16.5 (CAVITY_5)
- net IMU_SPI_MISO: now also J13.5 (D12 / PH8), J14.3 (CAVITY_3)
- net IMU_THUMB_CS_N: now also J13.3 (D10 / PA3), J15.1 (CAVITY_1), R18.2
- net IMU_THUMB_INT1: now also J12.6 (D5 / PE10), J16.1 (CAVITY_1)
- new net +3V3_IMU: R18.1, R19.1, R20.1, R21.1, R22.1
- new net IMU_SPI_MOSI: J14.5 (CAVITY_5)
- new net IMU_SPI_SCK: J14.1 (CAVITY_1)
- no-connect marks 4 -> 17
Other:
- note added: "CN7 DNC: pins 1,2,3,5,6. CN11 DNC: pins 1,2. CN12 DNC: pins 8 AREF, 9 SDA, 10 SCL."
- note added: "CN8-2 IOREF, CN8-4 3V3, CN8-5 5V, CN8-8 VIN: EXPLICIT NO-CONNECT. CN8-1 NC and CN8-3 RESET also DNC."
- note added: "CS PULL-UPS KEEP ALL IMUS DESELECTED WHILE DK IS OFF, RESETTING, BOOTING, HALTED, OR DISCONNECTED"
- note added: "DEFERRED PHYSICAL VALIDATION - NOT MEASURED"
- note added: "DK POSITIVE POWER PINS MUST NOT CONNECT TO PCB_GLOVE"
- note added: "ISM330DHCX INT1: active-high push-pull. MCU inputs: no internal pull. EXTI: thumb 10, index 5, middle 9, ring 0, pinky 11."
- note added: "J14 SPI cavities: 1 SCK, 2 GND, 3 MISO, 4 GND, 5 MOSI, 6 DNC / NO TERMINAL."
- note added: "J15 CS cavities: 1 THUMB, 2 GND, 3 INDEX, 4 MIDDLE, 5 RING, 6 PINKY."
- note added: "J16 INT cavities: 1 THUMB, 2 GND, 3 INDEX, 4 MIDDLE, 5 RING, 6 PINKY."
- note added: "NOT PHYSICALLY QUALIFIED / NOT WEARABLE QUALIFIED / NOT FOR FABRICATION"
- note added: "PCB_GLOVE POWERED THROUGH J9 EXTERNAL INPUT ONLY"
- note added: "R18-R22 = 10k to +3V3_IMU on glove side. PROVISIONAL - PHYSICAL RESET/BACKFEED VALIDATION REQUIRED."
- note added: "SPI5 initial firmware: MODE 3, IDLE HIGH, SOFTWARE NSS, 100 kHz-1 MHz. Final speed requires signal-integrity validation."
- note added: "STM32N6570-DK FOUR-CONNECTOR DIGITAL INTERFACE - DRAFT DEVELOPMENT HARDWARE"
- note removed: "+3V3_IMU is generated locally by the power-sheet LDO. Optional INT2 signals remain reserved but are not finally mapped."
- note removed: "All J1 numbers are logical drafting slots only; they do not correspond to CN4/CN7/CN8/CN11/CN12 physical positions."
- note removed: "Arduino and STMod+ signals may overlap. Solder bridges, voltage domains, on-board conflicts, EXTI capability, and reset states remain TBD."
- note removed: "DK +5 V IS NOT CONNECTED TO +5V_EXT — DK +3.3 V IS NOT CONNECTED TO +3V3_IMU"
- note removed: "DK AND PCB_glove SHARE GND ONLY THROUGH THE DOCUMENTED SIGNAL INTERFACE; POSITIVE POWER RAIL SLOTS ARE NO-CONNECTED."
- note removed: "DK_SPARE_TBD is intentionally no-connected; allocate only after the document-backed DK pin map."
- note removed: "DRAFT ONLY — J1 IS NOT A PHYSICAL DK CONNECTOR PINOUT"
- note removed: "Exact Arduino/STMod+/DK connector mapping requires local UM3300 and MB1939 schematic review."
- note removed: "STM32N6570-DK ADAPTER / HEADER LOGICAL INTERFACE"

Commit message: al
Parts:
- J14: value SPI HARNESS -> JST ZE SPI HARNESS [I]; footprint (none) -> PCB_glove:JST_ZE_BM06B-ZESS-TBT_1x06_P1.50mm_Vertical; symbol PCB_glove_Draft:HARNESS_1X6 -> PCB_glove_Draft:JST_ZE_BM06B_ZESS_TBT; CableLength (none) -> 50 mm preferred; 100 mm provisional maximum; CrimpTerminal 5055721200 -> SZE-002T-P0.3; FootprintStatus PROVISIONAL UNTIL PHASE 3 -> DIGITAL OVERLAY PASS; PHYSICAL QUALIFICATION OPEN; GroupLabel (none) -> J14 SPI ONLY [I]; HandTool 200218-4500 -> YRS-1460; MPN 5055750620 -> BM06B-ZESS-TBT; Manufacturer Molex -> JST; MatingHousing 5055700601 -> ZER-06V-S; Wire Alpha Wire 422607 -> Alpha Wire 422607, 26 AWG
- J15: value CS HARNESS -> JST ZE CS_N HARNESS [II]; footprint (none) -> PCB_glove:JST_ZE_BM06B-ZESS-TBT_1x06_P1.50mm_Vertical; symbol PCB_glove_Draft:HARNESS_1X6 -> PCB_glove_Draft:JST_ZE_BM06B_ZESS_TBT; CableLength (none) -> 50 mm preferred; 100 mm provisional maximum; CrimpTerminal 5055721200 -> SZE-002T-P0.3; FootprintStatus PROVISIONAL UNTIL PHASE 3 -> DIGITAL OVERLAY PASS; PHYSICAL QUALIFICATION OPEN; GroupLabel (none) -> J15 CS_N ONLY [II]; HandTool 200218-4500 -> YRS-1460; MPN 5055750620 -> BM06B-ZESS-TBT; Manufacturer Molex -> JST; MatingHousing 5055700601 -> ZER-06V-S; Wire Alpha Wire 422607 -> Alpha Wire 422607, 26 AWG
- J16: value INT HARNESS -> JST ZE INT1 HARNESS [III]; footprint (none) -> PCB_glove:JST_ZE_BM06B-ZESS-TBT_1x06_P1.50mm_Vertical; symbol PCB_glove_Draft:HARNESS_1X6 -> PCB_glove_Draft:JST_ZE_BM06B_ZESS_TBT; CableLength (none) -> 50 mm preferred; 100 mm provisional maximum; CrimpTerminal 5055721200 -> SZE-002T-P0.3; FootprintStatus PROVISIONAL UNTIL PHASE 3 -> DIGITAL OVERLAY PASS; PHYSICAL QUALIFICATION OPEN; GroupLabel (none) -> J16 INT1 ONLY [III]; HandTool 200218-4500 -> YRS-1460; MPN 5055750620 -> BM06B-ZESS-TBT; Manufacturer Molex -> JST; MatingHousing 5055700601 -> ZER-06V-S; Wire Alpha Wire 422607 -> Alpha Wire 422607, 26 AWG
Other:
- note added: "IDENTICAL JST ZE 6P PORTS: J14 SPI [I] / J15 CS_N [II] / J16 INT1 [III]. VERIFY GROUP. NO HOT-PLUG. PHYSICAL KEYING OPEN."
- note added: "J14 JST ZE SPI [I] circuits/cavities: 1 SCK, 2 GND, 3 MISO, 4 GND, 5 MOSI, 6 DNC / NO TERMINAL."
- note added: "J15 JST ZE CS_N [II] circuits/cavities: 1 THUMB, 2 GND, 3 INDEX, 4 MIDDLE, 5 RING, 6 PINKY."
- note added: "J16 JST ZE INT1 [III] circuits/cavities: 1 THUMB, 2 GND, 3 INDEX, 4 MIDDLE, 5 RING, 6 PINKY."
- note removed: "J14 SPI cavities: 1 SCK, 2 GND, 3 MISO, 4 GND, 5 MOSI, 6 DNC / NO TERMINAL."
- note removed: "J15 CS cavities: 1 THUMB, 2 GND, 3 INDEX, 4 MIDDLE, 5 RING, 6 PINKY."
- note removed: "J16 INT cavities: 1 THUMB, 2 GND, 3 INDEX, 4 MIDDLE, 5 RING, 6 PINKY."
- moved on the sheet: J14, J15, J16
Changed lines of the file:
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@@
     (pin "10")
   )
-  (symbol (lib_id "PCB_glove_Draft:HARNESS_1X6") (at 35.56 160.02 0) (unit 1)
-    (in_bom yes) (on_board yes)
-    (property "Reference" "J14" (at 35.56 148.57 0) (effects (font (size 1.27 1.27))))
-    (property "Value" "SPI HARNESS" (at 35.56 171.43 0) (effects (font (size 1.27 1.27))))
-    (property "Footprint" "" (at 35.56 173.97 0) (effects (font (size 1.27 1.27)) hide))
-    (property "Datasheet" "https://www.molex.com/en-us/products/part-detail/5055750620" (at 35.56 176.51 0) (effects (font (size 1.27 1.27)) hide))
-    (property "Manufacturer" "Molex" (at 35.56 160.02 0) (effects (font (size 1.27 1.27)) hide))
-    (property "MPN" "5055750620" (at 35.56 160.02 0) (effects (font (size 1.27 1.27)) hide))
-    (property "MatingHousing" "5055700601" (at 35.56 160.02 0) (effects (font (size 1.27 1.27)) hide))
-    (property "CrimpTerminal" "5055721200" (at 35.56 160.02 0) (effects (font (size 1.27 1.27)) hide))
-    (property "HandTool" "200218-4500" (at 35.56 160.02 0) (effects (font (size 1.27 1.27)) hide))
-    (property "Wire" "Alpha Wire 422607" (at 35.56 160.02 0) (effects (font (size 1.27 1.27)) hide))
-    (property "FootprintStatus" "PROVISIONAL UNTIL PHASE 3" (at 35.56 160.02 0) (effects (font (size 1.27 1.27)) hide))
+  (symbol (lib_id "PCB_glove_Draft:JST_ZE_BM06B_ZESS_TBT") (at 35.56 160.02 0) (unit 1)
+    (in_bom yes) (on_board yes)
+    (property "Reference" "J14" (at 35.56 142.24 0) (effects (font (size 1.27 1.27))))
+    (property "Value" "JST ZE SPI HARNESS [I]" (at 35.56 177.8 0) (effects (font (size 1.27 1.27))))
+    (property "Footprint" "PCB_glove:JST_ZE_BM06B-ZESS-TBT_1x06_P1.50mm_Vertical" (at 35.56 173.97 0) (effects (font (size 1.27 1.27)) hide))
+    (property "Datasheet" "https://www.jst-mfg.com/product/pdf/eng/eZE.pdf" (at 35.56 176.51 0) (effects (font (size 1.27 1.27)) hide))
+    (property "Manufacturer" "JST" (at 35.56 160.02 0) (effects (font (size 1.27 1.27)) hide))
+    (property "MPN" "BM06B-ZESS-TBT" (at 35.56 160.02 0) (effects (font (size 1.27 1.27)) hide))
+    (property "MatingHousing" "ZER-06V-S" (at 35.56 160.02 0) (effects (font (size 1.27 1.27)) hide))
+    (property "CrimpTerminal" "SZE-002T-P0.3" (at 35.56 160.02 0) (effects (font (size 1.27 1.27)) hide))
+    (property "HandTool" "YRS-1460" (at 35.56 160.02 0) (effects (font (size 1.27 1.27)) hide))
+    (property "Wire" "Alpha Wire 422607, 26 AWG" (at 35.56 160.02 0) (effects (font (size 1.27 1.27)) hide))
+    (property "FootprintStatus" "DIGITAL OVERLAY PASS; PHYSICAL QUALIFICATION OPEN" (at 35.56 160.02 0) (effects (font (size 1.27 1.27)) hide))
+    (property "CableLength" "50 mm preferred; 100 mm provisional maximum" (at 35.56 160.02 0) (effects (font (size 1.27 1.27)) hide))
+    (property "GroupLabel" "J14 SPI ONLY [I]" (at 35.56 160.02 0) (effects (font (size 1.27 1.27)) hide))
     (pin "1")
     (pin "2")
@@
     (pin "6")
   )
-  (symbol (lib_id "PCB_glove_Draft:HARNESS_1X6") (at 81.28 160.02 0) (unit 1)
-    (in_bom yes) (on_board yes)
-    (property "Reference" "J15" (at 81.28 148.57 0) (effects (font (size 1.27 1.27))))
-    (property "Value" "CS HARNESS" (at 81.28 171.43 0) (effects (font (size 1.27 1.27))))
-    (property "Footprint" "" (at 81.28 173.97 0) (effects (font (size 1.27 1.27)) hide))
-    (property "Datasheet" "https://www.molex.com/en-us/products/part-detail/5055750620" (at 81.28 176.51 0) (effects (font (size 1.27 1.27)) hide))
-    (property "Manufacturer" "Molex" (at 81.28 160.02 0) (effects (font (size 1.27 1.27)) hide))
-    (property "MPN" "5055750620" (at 81.28 160.02 0) (effects (font (size 1.27 1.27)) hide))
-    (property "MatingHousing" "5055700601" (at 81.28 160.02 0) (effects (font (size 1.27 1.27)) hide))
-    (property "CrimpTerminal" "5055721200" (at 81.28 160.02 0) (effects (font (size 1.27 1.27)) hide))
-    (property "HandTool" "200218-4500" (at 81.28 160.02 0) (effects (font (size 1.27 1.27)) hide))
-    (property "Wire" "Alpha Wire 422607" (at 81.28 160.02 0) (effects (font (size 1.27 1.27)) hide))
-    (property "FootprintStatus" "PROVISIONAL UNTIL PHASE 3" (at 81.28 160.02 0) (effects (font (size 1.27 1.27)) hide))
+  (symbol (lib_id "PCB_glove_Draft:JST_ZE_BM06B_ZESS_TBT") (at 81.28 160.02 0) (unit 1)
+    (in_bom yes) (on_board yes)
+    (property "Reference" "J15" (at 81.28 142.24 0) (effects (font (size 1.27 1.27))))
+    (property "Value" "JST ZE CS_N HARNESS [II]" (at 81.28 177.8 0) (effects (font (size 1.27 1.27))))
+    (property "Footprint" "PCB_glove:JST_ZE_BM06B-ZESS-TBT_1x06_P1.50mm_Vertical" (at 81.28 173.97 0) (effects (font (size 1.27 1.27)) hide))
+    (property "Datasheet" "https://www.jst-mfg.com/product/pdf/eng/eZE.pdf" (at 81.28 176.51 0) (effects (font (size 1.27 1.27)) hide))
+    (property "Manufacturer" "JST" (at 81.28 160.02 0) (effects (font (size 1.27 1.27)) hide))
+    (property "MPN" "BM06B-ZESS-TBT" (at 81.28 160.02 0) (effects (font (size 1.27 1.27)) hide))
+    (property "MatingHousing" "ZER-06V-S" (at 81.28 160.02 0) (effects (font (size 1.27 1.27)) hide))
+    (property "CrimpTerminal" "SZE-002T-P0.3" (at 81.28 160.02 0) (effects (font (size 1.27 1.27)) hide))
+    (property "HandTool" "YRS-1460" (at 81.28 160.02 0) (effects (font (size 1.27 1.27)) hide))
+    (property "Wire" "Alpha Wire 422607, 26 AWG" (at 81.28 160.02 0) (effects (font (size 1.27 1.27)) hide))
+    (property "FootprintStatus" "DIGITAL OVERLAY PASS; PHYSICAL QUALIFICATION OPEN" (at 81.28 160.02 0) (effects (font (size 1.27 1.27)) hide))
+    (property "CableLength" "50 mm preferred; 100 mm provisional maximum" (at 81.28 160.02 0) (effects (font (size 1.27 1.27)) hide))
+    (property "GroupLabel" "J15 CS_N ONLY [II]" (at 81.28 160.02 0) (effects (font (size 1.27 1.27)) hide))
     (pin "1")
     (pin "2")
@@
     (pin "6")
   )
-  (symbol (lib_id "PCB_glove_Draft:HARNESS_1X6") (at 127 160.02 0) (unit 1)
-    (in_bom yes) (on_board yes)
-    (property "Reference" "J16" (at 127 148.57 0) (effects (font (size 1.27 1.27))))
-    (property "Value" "INT HARNESS" (at 127 171.43 0) (effects (font (size 1.27 1.27))))
-    (property "Footprint" "" (at 127 173.97 0) (effects (font (size 1.27 1.27)) hide))
-    (property "Datasheet" "https://www.molex.com/en-us/products/part-detail/5055750620" (at 127 176.51 0) (effects (font (size 1.27 1.27)) hide))
-    (property "Manufacturer" "Molex" (at 127 160.02 0) (effects (font (size 1.27 1.27)) hide))
-    (property "MPN" "5055750620" (at 127 160.02 0) (effects (font (size 1.27 1.27)) hide))
-    (property "MatingHousing" "5055700601" (at 127 160.02 0) (effects (font (size 1.27 1.27)) hide))
-    (property "CrimpTerminal" "5055721200" (at 127 160.02 0) (effects (font (size 1.27 1.27)) hide))
-    (property "HandTool" "200218-4500" (at 127 160.02 0) (effects (font (size 1.27 1.27)) hide))
-    (property "Wire" "Alpha Wire 422607" (at 127 160.02 0) (effects (font (size 1.27 1.27)) hide))
-    (property "FootprintStatus" "PROVISIONAL UNTIL PHASE 3" (at 127 160.02 0) (effects (font (size 1.27 1.27)) hide))
+  (symbol (lib_id "PCB_glove_Draft:JST_ZE_BM06B_ZESS_TBT") (at 127 160.02 0) (unit 1)
+    (in_bom yes) (on_board yes)
+    (property "Reference" "J16" (at 127 142.24 0) (effects (font (size 1.27 1.27))))
+    (property "Value" "JST ZE INT1 HARNESS [III]" (at 127 177.8 0) (effects (font (size 1.27 1.27))))
+    (property "Footprint" "PCB_glove:JST_ZE_BM06B-ZESS-TBT_1x06_P1.50mm_Vertical" (at 127 173.97 0) (effects (font (size 1.27 1.27)) hide))
+    (property "Datasheet" "https://www.jst-mfg.com/product/pdf/eng/eZE.pdf" (at 127 176.51 0) (effects (font (size 1.27 1.27)) hide))
+    (property "Manufacturer" "JST" (at 127 160.02 0) (effects (font (size 1.27 1.27)) hide))
+    (property "MPN" "BM06B-ZESS-TBT" (at 127 160.02 0) (effects (font (size 1.27 1.27)) hide))
+    (property "MatingHousing" "ZER-06V-S" (at 127 160.02 0) (effects (font (size 1.27 1.27)) hide))
+    (property "CrimpTerminal" "SZE-002T-P0.3" (at 127 160.02 0) (effects (font (size 1.27 1.27)) hide))
+    (property "HandTool" "YRS-1460" (at 127 160.02 0) (effects (font (size 1.27 1.27)) hide))
+    (property "Wire" "Alpha Wire 422607, 26 AWG" (at 127 160.02 0) (effects (font (size 1.27 1.27)) hide))
+    (property "FootprintStatus" "DIGITAL OVERLAY PASS; PHYSICAL QUALIFICATION OPEN" (at 127 160.02 0) (effects (font (size 1.27 1.27)) hide))
+    (property "CableLength" "50 mm preferred; 100 mm provisional maximum" (at 127 160.02 0) (effects (font (size 1.27 1.27)) hide))
+    (property "GroupLabel" "J16 INT1 ONLY [III]" (at 127 160.02 0) (effects (font (size 1.27 1.27)) hide))
     (pin "1")
     (pin "2")
@@
     (effects (font (size 1.27 1.27)) (justify left bottom))
   )
-  (text "J14 SPI cavities: 1 SCK, 2 GND, 3 MISO, 4 GND, 5 MOSI, 6 DNC / NO TERMINAL." (at 15.24 195.58 0)
+  (text "J14 JST ZE SPI [I] circuits/cavities: 1 SCK, 2 GND, 3 MISO, 4 GND, 5 MOSI, 6 DNC / NO TERMINAL." (at 15.24 195.58 0)
     (effects (font (size 1.27 1.27)) (justify left bottom))
   )
-  (text "J15 CS cavities: 1 THUMB, 2 GND, 3 INDEX, 4 MIDDLE, 5 RING, 6 PINKY." (at 15.24 203.2 0)
+  (text "J15 JST ZE CS_N [II] circuits/cavities: 1 THUMB, 2 GND, 3 INDEX, 4 MIDDLE, 5 RING, 6 PINKY." (at 15.24 203.2 0)
     (effects (font (size 1.27 1.27)) (justify left bottom))
   )
-  (text "J16 INT cavities: 1 THUMB, 2 GND, 3 INDEX, 4 MIDDLE, 5 RING, 6 PINKY." (at 15.24 210.82 0)
+  (text "J16 JST ZE INT1 [III] circuits/cavities: 1 THUMB, 2 GND, 3 INDEX, 4 MIDDLE, 5 RING, 6 PINKY." (at 15.24 210.82 0)
     (effects (font (size 1.27 1.27)) (justify left bottom))
   )
+  (text "IDENTICAL JST ZE 6P PORTS: J14 SPI [I] / J15 CS_N [II] / J16 INT1 [III]. VERIFY GROUP. NO HOT-PLUG. PHYSICAL KEYING OPEN." (at 15.24 216.92 0)
+    (effects (font (size 1.27 1.27) (thickness 0.25)) (justify left bottom))
+  )
   (text "CS PULL-UPS KEEP ALL IMUS DESELECTED WHILE DK IS OFF, RESETTING, BOOTING, HALTED, OR DISCONNECTED" (at 15.24 220.98 0)
